File: board/spark.kicad_pcb (KiCad board)
At the start: 4 copper layers, 257 x 109 mm, 53 parts, among them J1 SFP+, J10 Conn_01x10, J2 SFP+, J3 SFP+, J4 SFP+, J5 SFP+, J6 SFP+, J7 PTH08T221W, J8 Conn_01x07_Male, J9 Conn_01x10, P1 CONN_02X20, P3 CONN_02X30, U1 XC3S50AN-TQG144, U2 AP3402

Commit message: Release 1.0
Parts:
- removed C1, C2, C3, C4: 100nF, Capacitor_SMD:C_0201_0603Metric
- removed C10, C12, C5, C6: 22uF, Capacitor_SMD:C_1210_3225Metric
- removed C11: 22pF, Capacitor_SMD:C_0201_0603Metric
- removed D1: ADM_LED, LED_SMD:LED_0201_0603Metric
- removed D2: ALARM_LED, LED_SMD:LED_0201_0603Metric
- removed J9: Conn_01x10, spark:sfp_header
- removed L1, L2: 4.7uH, Inductor_SMD:L_1210_3225Metric
- removed L3: 2.2uH, Inductor_SMD:L_1210_3225Metric
- removed R1, R4: R, Resistor_SMD:R_0201_0603Metric
- removed R10, R11: 150K, Resistor_SMD:R_0402_1005Metric
- removed R12, R13, R14, R16: 4K7, Resistor_SMD:R_0201_0603Metric
- removed R2, R3, R5, R6, R7: 10K, Resistor_SMD:R_0201_0603Metric
- removed R9: 100K, Resistor_SMD:R_0201_0603Metric
- removed the REF** at (186.0, 99.0)
- removed the REF** at (186.0, 154.0)
- removed the REF** at (100.0, 99.0)
- removed the REF** at (272.0, 99.0)
- removed U1: XC3S50AN-TQG144, Package_QFP:EQFP-144-1EP_20x20mm_P0.5mm_EP5x5mm
- removed U2: AP3402, Package_TO_SOT_SMD:TSOT-26-6
- added ?: , ice4pi:mount_hole, F.Cu at (163.0, 45.0)
- added ?: , ice4pi:mount_hole, F.Cu at (105.0, 45.0)
- added C101: 100nF, Capacitor_SMD:C_0402_1005Metric, B.Cu at (144.4, 124.7)
- added C102: 100nF, Capacitor_SMD:C_0402_1005Metric, B.Cu at (144.4, 108.5)
- added C103: 100nF, Capacitor_SMD:C_0402_1005Metric, B.Cu at (157.5, 111.0)
- added C104: 100nF, Capacitor_SMD:C_0402_1005Metric, B.Cu at (156.0, 111.0)
- added C105: 22uF, Capacitor_SMD:C_1210_3225Metric, B.Cu at (145.3, 119.2)
- added C106: 22uF, Capacitor_SMD:C_1210_3225Metric, B.Cu at (145.3, 114.0)
- added C201: 100nF, Capacitor_SMD:C_0402_1005Metric, B.Cu at (120.4, 124.7)
- added C202: 100nF, Capacitor_SMD:C_0402_1005Metric, B.Cu at (120.4, 108.5)
- added C203: 100nF, Capacitor_SMD:C_0402_1005Metric, B.Cu at (133.5, 111.0)
- added C204: 100nF, Capacitor_SMD:C_0402_1005Metric, B.Cu at (132.0, 111.0)
- added C205: 22uF, Capacitor_SMD:C_1210_3225Metric, B.Cu at (121.3, 119.2)
- added C206: 22uF, Capacitor_SMD:C_1210_3225Metric, B.Cu at (121.3, 114.0)
- added C301: 100nF, Capacitor_SMD:C_0402_1005Metric, B.Cu at (96.4, 124.7)
- added C302: 100nF, Capacitor_SMD:C_0402_1005Metric, B.Cu at (96.4, 108.5)
- added C303: 100nF, Capacitor_SMD:C_0402_1005Metric, B.Cu at (109.5, 111.0)
- added C304: 100nF, Capacitor_SMD:C_0402_1005Metric, B.Cu at (108.0, 111.0)
- added C305: 22uF, Capacitor_SMD:C_1210_3225Metric, B.Cu at (97.3, 119.2)
- added C306: 22uF, Capacitor_SMD:C_1210_3225Metric, B.Cu at (97.3, 114.0)
- added C401: 100nF, Capacitor_SMD:C_0402_1005Metric, B.Cu at (72.4, 124.7)
- added C402: 100nF, Capacitor_SMD:C_0402_1005Metric, B.Cu at (72.4, 108.5)
- added C403: 100nF, Capacitor_SMD:C_0402_1005Metric, B.Cu at (85.5, 111.0)
- added C404: 100nF, Capacitor_SMD:C_0402_1005Metric, B.Cu at (84.0, 111.0)
- added C405: 22uF, Capacitor_SMD:C_1210_3225Metric, B.Cu at (73.3, 119.2)
- added C406: 22uF, Capacitor_SMD:C_1210_3225Metric, B.Cu at (73.3, 114.0)
- added C501: 100nF, Capacitor_SMD:C_0402_1005Metric, B.Cu at (48.4, 124.7)
- added C502: 100nF, Capacitor_SMD:C_0402_1005Metric, B.Cu at (48.4, 108.5)
- added C503: 100nF, Capacitor_SMD:C_0402_1005Metric, B.Cu at (61.5, 111.0)
- added C504: 100nF, Capacitor_SMD:C_0402_1005Metric, B.Cu at (60.0, 111.0)
- added C505: 22uF, Capacitor_SMD:C_1210_3225Metric, B.Cu at (49.3, 119.2)
- added C506: 22uF, Capacitor_SMD:C_1210_3225Metric, B.Cu at (49.3, 114.0)
- added C601: 100nF, Capacitor_SMD:C_0402_1005Metric, B.Cu at (24.4, 124.7)
- added C602: 100nF, Capacitor_SMD:C_0402_1005Metric, B.Cu at (24.4, 108.5)
- added C603: 100nF, Capacitor_SMD:C_0402_1005Metric, B.Cu at (37.5, 111.0)
- added C604: 100nF, Capacitor_SMD:C_0402_1005Metric, B.Cu at (36.0, 111.0)
- added C605: 22uF, Capacitor_SMD:C_1210_3225Metric, B.Cu at (25.3, 119.2)
- added C606: 22uF, Capacitor_SMD:C_1210_3225Metric, B.Cu at (25.3, 114.0)
- added D101: ADM_LED, LED_SMD:LED_0402_1005Metric, F.Cu at (161.8, 104.2)
- added D102: ALARM_LED, LED_SMD:LED_0402_1005Metric, F.Cu at (152.2, 104.2)
- added D201: ADM_LED, LED_SMD:LED_0402_1005Metric, F.Cu at (137.8, 104.2)
- added D202: ALARM_LED, LED_SMD:LED_0402_1005Metric, F.Cu at (128.2, 104.2)
- added D301: ADM_LED, LED_SMD:LED_0402_1005Metric, F.Cu at (113.8, 104.2)
- added D302: ALARM_LED, LED_SMD:LED_0402_1005Metric, F.Cu at (104.2, 104.2)
- added D401: ADM_LED, LED_SMD:LED_0402_1005Metric, F.Cu at (89.8, 104.2)
- added D402: ALARM_LED, LED_SMD:LED_0402_1005Metric, F.Cu at (80.2, 104.2)
- added D501: ADM_LED, LED_SMD:LED_0402_1005Metric, F.Cu at (65.8, 104.2)
- added D502: ALARM_LED, LED_SMD:LED_0402_1005Metric, F.Cu at (56.2, 104.2)
- added D601: ADM_LED, LED_SMD:LED_0402_1005Metric, F.Cu at (41.8, 104.2)
- added D602: ALARM_LED, LED_SMD:LED_0402_1005Metric, F.Cu at (32.2, 104.2)
- added J109: Conn_01x10, spark:sfp_header, B.Cu at (157.0, 100.8)
- added J209: Conn_01x10, spark:sfp_header, B.Cu at (133.0, 100.8)
- added J309: Conn_01x10, spark:sfp_header, B.Cu at (109.0, 100.8)
- added J409: Conn_01x10, spark:sfp_header, B.Cu at (85.0, 100.8)
- added J509: Conn_01x10, spark:sfp_header, B.Cu at (61.0, 100.8)
- added J609: Conn_01x10, spark:sfp_header, B.Cu at (37.0, 100.8)
- added L101: 4.7uH, Inductor_SMD:L_1210_3225Metric, B.Cu at (145.3, 122.5)
- added L102: 4.7uH, Inductor_SMD:L_1210_3225Metric, B.Cu at (145.3, 110.7)
- added L201: 4.7uH, Inductor_SMD:L_1210_3225Metric, B.Cu at (121.3, 122.5)
- added L202: 4.7uH, Inductor_SMD:L_1210_3225Metric, B.Cu at (121.3, 110.7)
- added L301: 4.7uH, Inductor_SMD:L_1210_3225Metric, B.Cu at (97.3, 122.5)
- added L302: 4.7uH, Inductor_SMD:L_1210_3225Metric, B.Cu at (97.3, 110.7)
- added L401: 4.7uH, Inductor_SMD:L_1210_3225Metric, B.Cu at (73.3, 122.5)
- added L402: 4.7uH, Inductor_SMD:L_1210_3225Metric, B.Cu at (73.3, 110.7)
- added L501: 4.7uH, Inductor_SMD:L_1210_3225Metric, B.Cu at (49.3, 122.5)
- added L502: 4.7uH, Inductor_SMD:L_1210_3225Metric, B.Cu at (49.3, 110.7)
- added L601: 4.7uH, Inductor_SMD:L_1210_3225Metric, B.Cu at (25.3, 122.5)
- added L602: 4.7uH, Inductor_SMD:L_1210_3225Metric, B.Cu at (25.3, 110.7)
- added P2: Conn_02x20_Odd_Even, 96boards:Socket_Strip_SMD_2x20_Pitch2mm, F.Cu at (263.0, 90.0)
- added P4: Conn_02x20_Odd_Even, Connector_PinHeader_2.54mm:PinHeader_2x20_P2.54mm_Vertical_SMD, F.Cu at (134.0, 45.0)
- added P5: Conn_02x20_Odd_Even, Connector_PinHeader_2.54mm:PinHeader_2x20_P2.54mm_Vertical_SMD, F.Cu at (220.0, 45.0)
- added R101: 1K, Resistor_SMD:R_0402_1005Metric, F.Cu at (162.8, 104.2)
- added R102: 10K, Resistor_SMD:R_0402_1005Metric, F.Cu at (159.0, 70.5)
- added R103: 10K, Resistor_SMD:R_0402_1005Metric, F.Cu at (158.0, 70.5)
- added R104: 1K, Resistor_SMD:R_0402_1005Metric, F.Cu at (151.1, 104.2)
- added R105: 10K, Resistor_SMD:R_0402_1005Metric, F.Cu at (157.0, 70.5)
- added R106: 10K, Resistor_SMD:R_0402_1005Metric, B.Cu at (146.4, 124.7)
- added R107: 10K, Resistor_SMD:R_0402_1005Metric, B.Cu at (146.4, 108.5)
- added R201: 1K, Resistor_SMD:R_0402_1005Metric, F.Cu at (138.8, 104.2)
- added R202: 10K, Resistor_SMD:R_0402_1005Metric, F.Cu at (149.0, 70.5)
- added R203: 10K, Resistor_SMD:R_0402_1005Metric, F.Cu at (148.0, 70.5)
- added R204: 1K, Resistor_SMD:R_0402_1005Metric, F.Cu at (127.1, 104.2)
- added R205: 10K, Resistor_SMD:R_0402_1005Metric, F.Cu at (147.0, 70.5)
- added R206: 10K, Resistor_SMD:R_0402_1005Metric, B.Cu at (122.4, 124.7)
- added R207: 10K, Resistor_SMD:R_0402_1005Metric, B.Cu at (122.4, 108.5)
- added R301: 1K, Resistor_SMD:R_0402_1005Metric, F.Cu at (114.8, 104.2)
- added R302: 10K, Resistor_SMD:R_0402_1005Metric, F.Cu at (139.0, 70.5)
- added R303: 10K, Resistor_SMD:R_0402_1005Metric, F.Cu at (138.0, 70.5)
- added R304: 1K, Resistor_SMD:R_0402_1005Metric, F.Cu at (103.1, 104.2)
- added R305: 10K, Resistor_SMD:R_0402_1005Metric, F.Cu at (137.0, 70.5)
- added R306: 10K, Resistor_SMD:R_0402_1005Metric, B.Cu at (98.4, 124.7)
- added R307: 10K, Resistor_SMD:R_0402_1005Metric, B.Cu at (98.4, 108.5)
- added R401: 1K, Resistor_SMD:R_0402_1005Metric, F.Cu at (90.8, 104.2)
- added R402: 10K, Resistor_SMD:R_0402_1005Metric, F.Cu at (129.0, 70.5)
- added R403: 10K, Resistor_SMD:R_0402_1005Metric, F.Cu at (128.0, 70.5)
- added R404: 1K, Resistor_SMD:R_0402_1005Metric, F.Cu at (79.1, 104.2)
- added R405: 10K, Resistor_SMD:R_0402_1005Metric, F.Cu at (127.0, 70.5)
- added R406: 10K, Resistor_SMD:R_0402_1005Metric, B.Cu at (74.4, 124.7)
- added R407: 10K, Resistor_SMD:R_0402_1005Metric, B.Cu at (74.4, 108.5)
- added R501: 1K, Resistor_SMD:R_0402_1005Metric, F.Cu at (66.8, 104.2)
- added R502: 10K, Resistor_SMD:R_0402_1005Metric, F.Cu at (119.0, 70.5)
- added R503: 10K, Resistor_SMD:R_0402_1005Metric, F.Cu at (118.0, 70.5)
- added R504: 1K, Resistor_SMD:R_0402_1005Metric, F.Cu at (55.1, 104.2)
- added R505: 10K, Resistor_SMD:R_0402_1005Metric, F.Cu at (117.0, 70.5)
- added R506: 10K, Resistor_SMD:R_0402_1005Metric, B.Cu at (50.4, 124.7)
- added R507: 10K, Resistor_SMD:R_0402_1005Metric, B.Cu at (50.4, 108.5)
- added R601: 1K, Resistor_SMD:R_0402_1005Metric, F.Cu at (42.8, 104.2)
- added R602: 10K, Resistor_SMD:R_0402_1005Metric, F.Cu at (109.0, 70.5)
- added R603: 10K, Resistor_SMD:R_0402_1005Metric, F.Cu at (108.0, 70.5)
- added R604: 1K, Resistor_SMD:R_0402_1005Metric, F.Cu at (31.1, 104.2)
- added R605: 10K, Resistor_SMD:R_0402_1005Metric, F.Cu at (107.0, 70.5)
- added R606: 10K, Resistor_SMD:R_0402_1005Metric, B.Cu at (26.4, 124.7)
- added R607: 10K, Resistor_SMD:R_0402_1005Metric, B.Cu at (26.4, 108.5)
- added REF**: 96Boards CE Outline Brick Top, spark:96Boards_CE_outline_std_brick_top, B.Cu at (101.0, 95.0)
- added REF**: 96Boards CE Outline Brick Top, spark:96Boards_CE_outline_std_brick_top, B.Cu at (273.0, 95.0)
- added REF**: Hole_2.5MM, 96boards:Hole_2.5MM, F.Cu at (176.5, 59.5)
- added REF**: Hole_2.5MM, 96boards:Hole_2.5MM, F.Cu at (192.0, 59.5)
- added REF**: Hole_2.5MM, 96boards:Hole_2.5MM, F.Cu at (192.0, 91.0)
- added REF**: Hole_2.5MM, 96boards:Hole_2.5MM, F.Cu at (269.0, 91.0)
- ?, C7, C8, C9, J1, J2, J3, J4, J5, J6, P1, P3, R8: moved to F.Cu
- J10: value Conn_01x10 -> Barrel_Jack; footprint spark:sfp_header -> spark:PJ1-021-SMT-TR
- J7: footprint R-PDSS-B11 -> spark:R-PDSS-B11; moved to F.Cu
- J8: value Conn_01x07_Male -> Conn_02x30_Odd_Even; footprint Connector_PinHeader_2.00mm:PinHeader_1x07_P2.00mm_Vertical_SMD_Pin1Left -> Connector_PinHeader_2.00mm:PinHeader_2x30_P2.00mm_Vertical_SMD; moved to F.Cu
- REF** (x2): moved to B.Cu
- moved C7 322.5 mm to (25.2, 52.2)
- moved C8 313.5 mm to (29.8, 50.5)
- moved J7 307.0 mm to (33.0, 70.0)
- moved J6 299.0 mm to (37.0, 109.0)
- moved R8 285.0 mm to (44.0, 44.5), turned to 180 degrees
- moved C9 261.0 mm to (56.0, 52.0)
- moved J5 251.0 mm to (61.0, 109.0)
- moved J4 203.0 mm to (85.0, 109.0)
- moved REF** 173.0 mm to (273.0, 150.0), turned to 180 degrees
- moved REF** 171.0 mm to (101.0, 150.0), turned to 180 degrees
- moved J3 155.1 mm to (109.0, 109.0)
- moved P1 153.1 mm to (263.0, 101.0)
- moved J8 132.1 mm to (134.0, 76.6), turned to 270 degrees
- moved ? 120.8 mm to (58.5, 76.6), turned to 0 degrees
- moved P3 107.6 mm to (240.2, 134.6), turned to 180 degrees
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Connections:
- J1 pad 15: Net-(C3-Pad1) -> SFP0_VCC_T
- J1 pad 16: Net-(C4-Pad1) -> SFP0_VCC_R
- J1 pad 18: DSI_D1+ -> CSI1_C+
- J1 pad 19: DSI_D1- -> CSI1_C-
- J1 pad CAGE: Net-(J1-PadCAGE) -> CHASSIS
- J10 pad 1: I2C0_SCL -> SYS_DCIN
- J10 pad 2: I2C0_SDA -> GND
- J10 pad 3: GPIO_G -> GND
- J2 pad 1: Net-(J2-Pad1) -> GND
- J2 pad 10: Net-(J2-Pad10) -> GND
- J2 pad 11: Net-(J2-Pad10) -> GND
- J2 pad 14: Net-(J2-Pad10) -> GND
- J2 pad 15: Net-(J2-Pad15) -> SFP1_VCC_T
- J2 pad 16: Net-(J2-Pad16) -> SFP1_VCC_R
- J2 pad 17: Net-(J2-Pad1) -> GND
- J2 pad 2: Net-(J2-Pad2) -> SFP1_TX_FAULT
- J2 pad 20: Net-(J2-Pad1) -> GND
- J2 pad 3: Net-(J2-Pad3) -> SFP1_TX_DISABLE
- J2 pad 4: Net-(J2-Pad4) -> SFP1_SDA
- J2 pad 5: Net-(J2-Pad5) -> SFP1_SCL
- J2 pad 6: Net-(J2-Pad6) -> SFP1_MOD_ABS
- J2 pad 7: Net-(J2-Pad7) -> SFP1_RS0
- J2 pad 8: Net-(J2-Pad8) -> SFP1_RX_LOS
- J2 pad 9: Net-(J2-Pad9) -> SFP1_RS1
- J2 pad CAGE: Net-(J2-PadCAGE) -> CHASSIS
- J3 pad 1: Net-(J3-Pad1) -> GND
- J3 pad 10: Net-(J3-Pad10) -> GND
- J3 pad 11: Net-(J3-Pad10) -> GND
- J3 pad 12: CSI1_C- -> DSI_D1-
- J3 pad 13: CSI1_C+ -> DSI_D1+
- J3 pad 14: Net-(J3-Pad10) -> GND
- J3 pad 15: Net-(J3-Pad15) -> SFP2_VCC_T
- J3 pad 16: Net-(J3-Pad16) -> SFP2_VCC_R
- J3 pad 17: Net-(J3-Pad1) -> GND
- J3 pad 2: Net-(J3-Pad2) -> SFP2_TX_FAULT
- J3 pad 20: Net-(J3-Pad1) -> GND
- J3 pad 3: Net-(J3-Pad3) -> SFP2_TX_DISABLE
- J3 pad 4: Net-(J3-Pad4) -> SFP2_SDA
- J3 pad 5: Net-(J3-Pad5) -> SFP2_SCL
- J3 pad 6: Net-(J3-Pad6) -> SFP2_MOD_ABS
- J3 pad 7: Net-(J3-Pad7) -> SFP2_RS0
- J3 pad 8: Net-(J3-Pad8) -> SFP2_RX_LOS
- J3 pad 9: Net-(J3-Pad9) -> SFP2_RS1
- J3 pad CAGE: Net-(J3-PadCAGE) -> CHASSIS
- J4 pad 1: Net-(J4-Pad1) -> GND
- J4 pad 10: Net-(J4-Pad10) -> GND
- J4 pad 11: Net-(J4-Pad10) -> GND
- J4 pad 12: CSI1_D0- -> DSI_CLK-
- J4 pad 13: CSI1_D0+ -> DSI_CLK+
- J4 pad 14: Net-(J4-Pad10) -> GND
- J4 pad 15: Net-(J4-Pad15) -> SFP3_VCC_T
- J4 pad 16: Net-(J4-Pad16) -> SFP3_VCC_R
- J4 pad 17: Net-(J4-Pad1) -> GND
- J4 pad 18: CSI0_D3+ -> CSI1_D0+
- J4 pad 19: CSI0_D3- -> CSI1_D0-
- J4 pad 2: Net-(J4-Pad2) -> SFP3_TX_FAULT
- J4 pad 20: Net-(J4-Pad1) -> GND
- J4 pad 3: Net-(J4-Pad3) -> SFP3_TX_DISABLE
- J4 pad 4: Net-(J4-Pad4) -> SFP3_SDA
- J4 pad 5: Net-(J4-Pad5) -> SFP3_SCL
- J4 pad 6: Net-(J4-Pad6) -> SFP3_MOD_ABS
- J4 pad 7: Net-(J4-Pad7) -> SFP3_RS0
- J4 pad 8: Net-(J4-Pad8) -> SFP3_RX_LOS
- J4 pad 9: Net-(J4-Pad9) -> SFP3_RS1
- J4 pad CAGE: Net-(J4-PadCAGE) -> CHASSIS
- J5 pad 1: Net-(J5-Pad1) -> GND
- J5 pad 10: Net-(J5-Pad10) -> GND
- J5 pad 11: Net-(J5-Pad10) -> GND
- J5 pad 14: Net-(J5-Pad10) -> GND
- J5 pad 15: Net-(J5-Pad15) -> SFP4_VCC_T
- J5 pad 16: Net-(J5-Pad16) -> SFP4_VCC_R
- J5 pad 17: Net-(J5-Pad1) -> GND
- J5 pad 2: Net-(J5-Pad2) -> SFP4_TX_FAULT
- J5 pad 20: Net-(J5-Pad1) -> GND
- J5 pad 3: Net-(J5-Pad3) -> SFP4_TX_DISABLE
- J5 pad 4: Net-(J5-Pad4) -> SFP4_SDA
- J5 pad 5: Net-(J5-Pad5) -> SFP4_SCL
- J5 pad 6: Net-(J5-Pad6) -> SFP4_MOD_ABS
- J5 pad 7: Net-(J5-Pad7) -> SFP4_RS0
- J5 pad 8: Net-(J5-Pad8) -> SFP4_RX_LOS
- J5 pad 9: Net-(J5-Pad9) -> SFP4_RS1
- J5 pad CAGE: Net-(J5-PadCAGE) -> CHASSIS
- J6 pad 1: Net-(J6-Pad1) -> GND
- J6 pad 10: Net-(J6-Pad10) -> GND
- J6 pad 11: Net-(J6-Pad10) -> GND
- J6 pad 12: CSI0_D0- -> CSI0_D3-
- J6 pad 13: CSI0_D0+ -> CSI0_D3+
- J6 pad 14: Net-(J6-Pad10) -> GND
- J6 pad 15: Net-(J6-Pad15) -> SFP5_VCC_T
- J6 pad 16: Net-(J6-Pad16) -> SFP5_VCC_R
- J6 pad 17: Net-(J6-Pad1) -> GND
- J6 pad 2: Net-(J6-Pad2) -> SFP5_TX_FAULT
- J6 pad 20: Net-(J6-Pad1) -> GND
- J6 pad 3: Net-(J6-Pad3) -> SFP5_TX_DISABLE
- J6 pad 4: Net-(J6-Pad4) -> SFP5_SDA
- J6 pad 5: Net-(J6-Pad5) -> SFP5_SCL
- J6 pad 6: Net-(J6-Pad6) -> SFP5_MOD_ABS
- J6 pad 7: Net-(J6-Pad7) -> SFP5_RS0
- J6 pad 8: Net-(J6-Pad8) -> SFP5_RX_LOS
- J6 pad 9: Net-(J6-Pad9) -> SFP5_RS1
- J6 pad CAGE: Net-(J6-PadCAGE) -> CHASSIS
- J8 pad 1: +3V3 -> SFP0_ADM_LED
- J8 pad 2: GND -> SFP0_RS1
- J8 pad 3: JTAG_TCK -> SFP0_RX_LOS
- J8 pad 4: JTAG_TMS -> SFP0_RS0
- J8 pad 5: JTAG_TDI -> SFP0_MOD_ABS
- J8 pad 6: Net-(J8-Pad6) -> SFP0_SCL
- J8 pad 7: JTAG_TDO -> SFP0_SDA
- REF** pad 1: GND -> CHASSIS (x2)
Routing:
- net GND: track 237.0 -> 1343.0 mm, vias 35 -> 110
- net +5V: track 320.3 -> 25.3 mm
- net SYS_DCIN: track 345.7 -> 75.6 mm, vias 0 -> 7
- net CSI0_D0+: track 246.0 -> 0.00 mm
- net CSI0_D0-: track 244.5 -> 0.00 mm
- net +1V8: track 233.3 -> 14.3 mm
- net CHASSIS: track 0.00 -> 202.4 mm
- net DSI_CLK+: track 0.00 -> 189.5 mm, vias 0 -> 2
- net DSI_CLK-: track 0.00 -> 188.2 mm, vias 0 -> 2
- net Net-(P4-Pad40): track 0.00 -> 155.2 mm, vias 0 -> 2
- net Net-(P4-Pad38): track 0.00 -> 152.9 mm, vias 0 -> 2
- net Net-(P4-Pad36): track 0.00 -> 150.6 mm, vias 0 -> 2
- net Net-(P4-Pad32): track 0.00 -> 145.9 mm, vias 0 -> 2
- net Net-(P4-Pad28): track 0.00 -> 140.2 mm, vias 0 -> 2
- net Net-(P4-Pad26): track 0.00 -> 137.9 mm, vias 0 -> 2
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- added copper zone on F.Cu, net +3V3
- added copper zone on In2.Cu, net +3V3
- added copper zone on In2.Cu, net SYS_DCIN
- removed copper zone on B.Cu, net GND
- removed copper zone on In2.Cu, net GND
Other:
- board text added: "Version: spark-1"
- board text removed: "Version: spark-0"

Commit message: Release 2.0
Parts:
- removed the REF** at (273.0, 95.0)
- removed the REF** at (176.5, 59.5)
- removed the REF** at (192.0, 59.5)
- removed the REF** at (192.0, 91.0)
- removed the REF** at (269.0, 91.0)
- added ?: , spark:mount_hole, F.Cu at (192.0, 45.0)
- added ?: , spark:mount_hole, F.Cu at (250.0, 45.0)
- added P6: CONN_02X30, spark:5177983-2, F.Cu at (240.2, 55.5)
- added REF**: stencil_hole_3mm, spark:stencil_hole_3mm, F.Cu at (20.0, 53.0)
- added REF**: 96Boards CE Outline Brick, spark:96Boards_CE_outline_std_brick, F.Cu at (273.0, 41.0)
- added REF**: Hole_2.5MM, spark:Hole_2.5MM, F.Cu at (269.0, 45.0)
- added REF**: stencil_hole_3mm, spark:stencil_hole_3mm, F.Cu at (20.0, 138.0)
- added SW1: SW_Push, Button_Switch_THT:SW_Tactile_SPST_Angled_PTS645Vx83-2LFS, F.Cu at (179.0, 147.0)
- added SW2: SW_DIP_x06, Button_Switch_SMD:SW_DIP_SPSTx06_Slide_Omron_A6H-6101_W6.15mm_P1.27mm, F.Cu at (108.0, 58.0)
- ? (x2): footprint ice4pi:mount_hole -> spark:mount_hole
- P1: footprint 96boards:Pin_Header_SMD_2x20_Pitch2mm -> spark:Pin_Header_SMD_2x20_Pitch2mm
- P2: footprint 96boards:Socket_Strip_SMD_2x20_Pitch2mm -> spark:Socket_Strip_SMD_2x20_Pitch2mm
- P3: footprint 96boards:61083-063400LF -> spark:61083-063400LF
- REF**: footprint 96boards:96Boards_CE_outline_std -> spark:96Boards_CE_outline_std
- moved ? 1.00 mm to (164.0, 45.0)
- moved ? 1.00 mm to (106.0, 45.0)
- moved P4 1.00 mm to (135.0, 45.0)
- moved P5 1.00 mm to (221.0, 45.0)
Connections:
- REF** pad 1: CHASSIS -> (no net)
Routing:
- net PWR_BTN_N: track 6.96 -> 145.6 mm
- net USB_D+: track 0.00 -> 116.8 mm, vias 0 -> 2
- net USB_D-: track 0.00 -> 113.5 mm, vias 0 -> 2
- net HSIC_STR: track 0.00 -> 95.4 mm, vias 0 -> 4
- net HSIC_DATA: track 0.00 -> 95.4 mm, vias 0 -> 4
- net CLK0/CSI0_MCLK: track 0.00 -> 93.0 mm, vias 0 -> 2
- net CLK1/CSI1_MCLK: track 0.00 -> 92.8 mm, vias 0 -> 2
- net SD_DAT3/SPI1_CS: track 0.00 -> 92.5 mm, vias 0 -> 2
- net SD_SCLK/SPI1_SCLK: track 0.00 -> 92.5 mm, vias 0 -> 2
- net SD_DAT2: track 0.00 -> 92.5 mm, vias 0 -> 2
- net SD_DAT1: track 0.00 -> 92.5 mm, vias 0 -> 2
- net SD_CMD/SPI1_DIN: track 0.00 -> 92.5 mm, vias 0 -> 2
- net SD_DAT0/SPI1_DOUT: track 0.00 -> 92.5 mm, vias 0 -> 2
- net I2C3_SDA: track 0.00 -> 74.7 mm, vias 0 -> 2
- net I2C3_SCL: track 0.00 -> 74.7 mm, vias 0 -> 2
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Other:
- board text added: "1"
- board text added: ":"
- board text added: "P/N"
- board text added: "REV"
- board text added: "SPARK-V2"
- board text removed: "Version: spark-1"

Commit message: Release 2.0-2
Parts:
- removed the REF** at (273.0, 41.0)
- moved REF** 2.50 mm to (20.0, 50.5)
- moved REF** 2.50 mm to (20.0, 140.5)
- moved P6 1.00 mm to (240.2, 56.5)
Connections:
- P4 pad 5: GND -> Net-(P4-Pad5)
- P4 pad 6: Net-(P4-Pad6) -> GND
- P5 pad 5: GND -> Net-(P4-Pad5)
- P5 pad 6: Net-(P4-Pad6) -> GND
- REF** pad 1: (no net) -> CHASSIS
Routing:
- net Net-(P4-Pad6): track 108.3 -> 0.00 mm, vias 2 -> 0
- net Net-(P4-Pad5): track 0.00 -> 99.7 mm, vias 0 -> 2
- net GND: track 1412.4 -> 1421.8 mm
- net HSIC_DATA: track 95.4 -> 93.4 mm
- net HSIC_STR: track 95.4 -> 93.4 mm
- net CLK0/CSI0_MCLK: track 93.0 -> 91.8 mm
- net SD_DAT3/SPI1_CS: track 92.5 -> 91.5 mm
- net SD_SCLK/SPI1_SCLK: track 92.5 -> 91.5 mm
- net SD_DAT2: track 92.5 -> 91.5 mm
- net SD_DAT1: track 92.5 -> 91.5 mm
- net SD_DAT0/SPI1_DOUT: track 92.5 -> 91.5 mm
- net SD_CMD/SPI1_DIN: track 92.5 -> 91.5 mm
- net I2C3_SDA: track 74.7 -> 73.7 mm
- net I2C3_SCL: track 74.7 -> 73.7 mm
- net I2C2_SDA: track 74.7 -> 73.7 mm
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
Commit message: Release 2.0-3
Parts:
- added REF**: 96Boards CE Outline Brick, spark:96Boards_CE_outline_std_brick, B.Cu at (188.0, 41.0)
Other:
- board text added: "3"
- board text removed: "1"
Changed lines of the file:
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@@
     (tracks 3350)
     (zones 0)
-    (modules 140)
+    (modules 141)
     (nets 228)
   )
   (page A4)
   (title_block
-    (title "Spark v.2, rev.2, (96Boards extension connector 6x SFP+)")
-    (date 2020-07-15)
+    (title "Spark v.2, rev.3, (96Boards extension connector 6x SFP+)")
+    (date 2020-10-28)
     (rev A)
     (company "Lightside Instruments AS")
@@
     (uvia_drill 0.1)
   )
+  (module spark:96Boards_CE_outline_std_brick (layer B.Cu)
+    (at 188 41)
+    (descr "module 1 pin (ou trou mecanique de percage)")
+    (tags "96Boards, formfactor, mezzanine")
+    (fp_text reference REF** (at 2.5 -1) (layer F.Fab) hide
+      (effects (font (size 1 1) (thickness 0.15)))
+    )
+    (fp_text value "96Boards CE Outline Brick" (at 42.5 -1.5) (layer F.Fab) hide
+      (effects (font (size 1 1) (thickness 0.15)))
+    )
+    (fp_line (start 85 54) (end 85 0) (layer F.Fab) (width 0.15))
+    (fp_circle (center 81 50) (end 83.6 50) (layer B.CrtYd) (width 0.05))
+    (fp_circle (center 4 50) (end 6.6 50) (layer B.CrtYd) (width 0.05))
+    (fp_circle (center 81 50) (end 83 49.2) (layer B.Fab) (width 0.1))
+    (fp_circle (center 4 50) (end 6 49.2) (layer B.Fab) (width 0.1))
+    (fp_circle (center 81 18.5) (end 83.6 18.5) (layer B.CrtYd) (width 0.05))
+    (fp_circle (center 81 18.5) (end 83 17.7) (layer B.Fab) (width 0.1))
+    (fp_circle (center 4 18.5) (end 6.6 18.5) (layer B.CrtYd) (width 0.05))
+    (fp_circle (center 4 18.5) (end 6 17.7) (layer B.Fab) (width 0.1))
+    (fp_line (start 0 0) (end 0 54) (layer F.Fab) (width 0.15))
+    (fp_line (start 0 54) (end 85 54) (layer F.Fab) (width 0.15))
+    (fp_line (start 85 0) (end 0 0) (layer F.Fab) (width 0.15))
+    (pad 1 thru_hole circle (at 81 50) (size 4.5 4.5) (drill 2.7) (layers *.Cu *.Mask))
+    (pad 1 thru_hole circle (at 4 50) (size 4.5 4.5) (drill 2.7) (layers *.Cu *.Mask))
+    (pad 1 thru_hole circle (at 81 18.5) (size 4.5 4.5) (drill 2.7) (layers *.Cu *.Mask))
+    (pad 1 thru_hole circle (at 4 18.5) (size 4.5 4.5) (drill 2.7) (layers *.Cu *.Mask))
+  )
   (module spark:stencil_hole_3mm (layer F.Cu)
     (at 20 50.5)
@@
     )
   )
-  (gr_text 1 (at 74.5 64.9) (layer F.Cu)
+  (gr_text 3 (at 74.5 64.9) (layer F.Cu)
     (effects (font (size 1.5 1.5) (thickness 0.3)))
   )
@@
       (pts
         (xy 273.7 97.2) (xy 265.7 97.2) (xy 265.7 97.18374) (xy 224.5 97.1) (xy 224.5 93.7)
-        (xy 265 93.8) (xy 265 45.7) (xy 74.3 45.6) (xy 74.3 54.3) (xy 69.3 54.3)
-        (xy 69.3 45.6) (xy 15.7 45.6) (xy 15.7 40.4) (xy 265.7 40.303101) (xy 265.7 40.3)
-        (xy 273.7 40.3)
+        (xy 265 93.8) (xy 265 80) (xy 260 80) (xy 260 45.7) (xy 74.3 45.6)
+        (xy 74.3 54.3) (xy 69.3 54.3) (xy 69.3 45.6) (xy 15.7 45.6) (xy 15.7 40.4)
+        (xy 265.7 40.303101) (xy 265.7 40.3) (xy 273.7 40.3)
       )
     )

Commit message: Release 2.0-4
Parts:
- C105, C106, C205, C206, C305, C306, C405, C406, C505, C506, C605, C606, C8: footprint Capacitor_SMD:C_1210_3225Metric -> Diode_SMD:D_1210_3225Metric
- moved J7 15.3 mm to (43.0, 58.4)
Other:
- board text added: "4"
- board text removed: "3"

Commit message: Release 2.0-5
Connections:
- P4 pad 1: Net-(P4-Pad1) -> +3V3
- P4 pad 17: Net-(P4-Pad17) -> +3V3
- P5 pad 1: Net-(P4-Pad1) -> +3V3
- P5 pad 17: Net-(P4-Pad17) -> +3V3
Routing:
- net +3V3: track 138.8 -> 354.1 mm, vias 46 -> 55
- net Net-(P4-Pad17): track 116.9 -> 0.00 mm, vias 2 -> 0
- net Net-(P4-Pad1): track 95.7 -> 0.00 mm, vias 2 -> 0
- net GND: track 1421.8 -> 1459.9 mm, vias 120 -> 147

Commit message: Release 2.0-6
Parts:
- added SW3: SW_DIP_x01, Connector_PinHeader_2.54mm:PinHeader_1x02_P2.54mm_Vertical, F.Cu at (30.8, 56.4)
- moved REF** 70.0 mm to (20.0, 120.5)
- moved C7 36.0 mm to (60.0, 61.5), turned to 90 degrees
- moved C8 28.8 mm to (55.5, 63.2), turned to 90 degrees
Routing:
- net GND: track 1459.9 -> 1489.1 mm, vias 147 -> 146
- net SYS_DCIN: track 62.5 -> 90.5 mm, vias 5 -> 4
- net Net-(J7-Pad11): track 0.00 -> 7.61 mm
- net +3V3: vias 55 -> 56
- added copper zone on F.Cu, net GND
Other:
- board text added: "6"
- board text removed: "4"

Commit message: Release 2.0-7
Parts:
- added C1: C, Capacitor_SMD:C_0402_1005Metric, F.Cu at (70.2, 49.5)
- added R1: 13K3, Capacitor_SMD:C_0402_1005Metric, F.Cu at (67.7, 46.9)
- added R2: 10K, Capacitor_SMD:C_0402_1005Metric, F.Cu at (70.2, 51.8)
- added SW4: SW_DIP_x01, Connector_PinHeader_2.54mm:PinHeader_1x02_P2.54mm_Vertical, F.Cu at (64.5, 58.7)
- added U1: LTM4624IYPBF, spark:Analog_Devices_Inc-BGA-0-05-08-1905_Rev_C-0, F.Cu at (65.9, 51.3)
Connections:
- net Net-(J7-Pad11) renamed INHIBIT_3V3
Routing:
- net SYS_DCIN: track 90.5 -> 132.2 mm, vias 4 -> 8
- net GND: track 1489.1 -> 1507.3 mm, vias 146 -> 152
- net Net-(R2-Pad1): track 0.00 -> 11.2 mm, vias 0 -> 1
- net Net-(U1-PadC4): track 0.00 -> 3.10 mm
- net Net-(R1-Pad1): track 0.00 -> 1.94 mm
- net Net-(C1-Pad1): track 0.00 -> 1.78 mm
- added copper zone on F.Cu, net SYS_DCIN
Other:
- board text added: "7"
- board text removed: "6"
