File: board/spark.kicad_pcb (KiCad board)
At the start: 4 copper layers, 257 x 109 mm, 147 parts, among them J1 SFP+, J10 Barrel_Jack, J109 Conn_01x10, J2 SFP+, J209 Conn_01x10, J3 SFP+, J309 Conn_01x10, J4 SFP+, J409 Conn_01x10, J5 SFP+, J509 Conn_01x10, J6 SFP+, J609 Conn_01x10, J7 PTH08T221W, J8 Conn_02x30_Odd_Even, P1 CONN_02X20, P2 Conn_02x20_Odd_Even, P3 CONN_02X30, P4 Conn_02x20_Odd_Even, P5 Conn_02x20_Odd_Even, P6 CONN_02X30, SW1 SW_Push, SW2 SW_DIP_x06, SW3 SW_DIP_x01, SW4 SW_DIP_x01, U1 LTM4624IYPBF

Commit message: Release 2.0-8
Parts:
- P4, P5: footprint Connector_PinHeader_2.54mm:PinHeader_2x20_P2.54mm_Vertical_SMD -> spark:PinHeader_2x20_P2.54mm_Vertical_SMD_Alignment_Pin
Connections:
- net INHIBIT_3V3 renamed Net-(J7-Pad11)
- J7 pad 9: Net-(J7-Pad9) -> (no net)
- P3 pad 10: CSI0_D0- -> (no net)
- P3 pad 60: Net-(P3-Pad60) -> (no net)
- P3 pad 8: CSI0_D0+ -> (no net)
- P6 pad 10: Net-(P6-Pad10) -> (no net)
- P6 pad 14: Net-(P6-Pad14) -> (no net)
- P6 pad 16: Net-(P6-Pad16) -> (no net)
- P6 pad 2: Net-(P6-Pad2) -> (no net)
- P6 pad 20: Net-(P6-Pad20) -> (no net)
- P6 pad 21: Net-(P6-Pad21) -> (no net)
- P6 pad 22: Net-(P6-Pad22) -> (no net)
- P6 pad 23: Net-(P6-Pad23) -> (no net)
- P6 pad 26: Net-(P6-Pad26) -> (no net)
- P6 pad 27: Net-(P6-Pad27) -> (no net)
- P6 pad 28: Net-(P6-Pad28) -> (no net)
- P6 pad 29: Net-(P6-Pad29) -> (no net)
- P6 pad 33: Net-(P6-Pad33) -> (no net)
- P6 pad 35: Net-(P6-Pad35) -> (no net)
- P6 pad 39: Net-(P6-Pad39) -> (no net)
- P6 pad 4: Net-(P6-Pad4) -> (no net)
- P6 pad 41: Net-(P6-Pad41) -> (no net)
- P6 pad 42: Net-(P6-Pad42) -> (no net)
- P6 pad 44: Net-(P6-Pad44) -> (no net)
- P6 pad 45: Net-(P6-Pad45) -> (no net)
- P6 pad 47: Net-(P6-Pad47) -> (no net)
- P6 pad 48: Net-(P6-Pad48) -> (no net)
- P6 pad 50: Net-(P6-Pad50) -> (no net)
- P6 pad 54: Net-(P6-Pad54) -> (no net)
- P6 pad 56: Net-(P6-Pad56) -> (no net)
- P6 pad 60: Net-(P6-Pad60) -> (no net)
- P6 pad 8: Net-(P6-Pad8) -> (no net)
- U1 pad A1: Net-(U1-PadA1) -> (no net)
- U1 pad A4: Net-(U1-PadA4) -> (no net)
- U1 pad A5: Net-(U1-PadA5) -> (no net)
- U1 pad B2: Net-(U1-PadB2) -> (no net)
- U1 pad B5: Net-(U1-PadB5) -> (no net)
- U1 pad C2: Net-(U1-PadC2) -> (no net)
Routing:
- net GND: track 1507.3 -> 1500.6 mm, vias 152 -> 151
- net Net-(P4-Pad3): track 97.7 -> 92.6 mm
- net Net-(P4-Pad2): track 105.7 -> 107.9 mm
- net Net-(P4-Pad38): track 150.0 -> 148.4 mm, vias 2 -> 4
Other:
- board text added: "8"
- board text removed: "7"

Commit message: Release 2.0-9
Parts:
- added R3: 4K7, Resistor_SMD:R_0402_1005Metric, F.Cu at (231.5, 84.1)
- added R4: 4K7, Resistor_SMD:R_0402_1005Metric, F.Cu at (230.2, 84.1)
- added R5: 200K, Resistor_SMD:R_0402_1005Metric, F.Cu at (227.7, 74.5)
- added R6: 4K7, Resistor_SMD:R_0402_1005Metric, F.Cu at (230.2, 74.5)
- added R7: 4K7, Resistor_SMD:R_0402_1005Metric, F.Cu at (231.5, 74.5)
- added U2: PCA9306, Package_SO:SO-8_3.9x4.9mm_P1.27mm, F.Cu at (229.6, 79.3)
Connections:
- net Net-(P4-Pad3) renamed RPI_I2C_SDA
- net Net-(P4-Pad5) renamed RPI_I2C_SCL
Routing:
- net RPI_I2C_SDA: track 92.6 -> 144.6 mm, vias 2 -> 4
- net RPI_I2C_SCL: track 99.7 -> 151.2 mm, vias 2 -> 4
- net I2C0_SCL: track 14.6 -> 40.2 mm
- net I2C0_SDA: track 14.6 -> 35.8 mm
- net +1V8: track 15.2 -> 23.8 mm
- net GND: track 1500.6 -> 1508.2 mm
- net +3V3: track 354.1 -> 359.2 mm, vias 56 -> 57
- net Net-(R5-Pad2): track 0.00 -> 3.01 mm
Other:
- board text added: "9"
- board text removed: "8"

Commit message: spark-pdu-1.0-1
Parts:
- removed the ? at (164.0, 45.0)
- removed the ? at (106.0, 45.0)
- removed C1: C, Capacitor_SMD:C_0402_1005Metric
- removed C101, C102, C103, C104, C201, C202, C203, C204, C301, C302, C303, C304, C401, C402, C403, C404, C501, C502, C503, C504, C601, C602, C603, C604: 100nF, Capacitor_SMD:C_0402_1005Metric
- removed C105, C106, C205, C206, C305, C306, C405, C406, C505, C506, C605, C606, C8: 22uF, Diode_SMD:D_1210_3225Metric
- removed C7: 330uF, Capacitor_Tantalum_SMD:CP_EIA-7343-31_Kemet-D
- removed C9: 220uF, Capacitor_Tantalum_SMD:CP_EIA-7343-31_Kemet-D
- removed D102, D202, D302, D402, D502, D602: ALARM_LED, LED_SMD:LED_0402_1005Metric
- removed J109, J209, J309, J409, J509, J609: Conn_01x10, spark:sfp_header
- removed J3, J4, J5, J6: SFP+, spark:molex-sfp-plus-747540-101
- removed J7: PTH08T221W, spark:R-PDSS-B11
- removed J8: Conn_02x30_Odd_Even, Connector_PinHeader_2.00mm:PinHeader_2x30_P2.00mm_Vertical_SMD
- removed L101, L102, L201, L202, L301, L302, L401, L402, L501, L502, L601, L602: 4.7uH, Inductor_SMD:L_1210_3225Metric
- removed P3: CONN_02X30, spark:61083-063400LF
- removed P4, P5: Conn_02x20_Odd_Even, spark:PinHeader_2x20_P2.54mm_Vertical_SMD_Alignment_Pin
- removed P6: CONN_02X30, spark:5177983-2
- removed R1: 13K3, Capacitor_SMD:C_0402_1005Metric
- removed R103, R105, R106, R107, R203, R205, R206, R207, R303, R305, R306, R307, R403, R405, R406, R407, R503, R505, R506, R507, R603, R605, R606, R607: 10K, Resistor_SMD:R_0402_1005Metric
- removed R104, R204, R304, R404, R504, R604: 1K, Resistor_SMD:R_0402_1005Metric
- removed R2: 10K, Capacitor_SMD:C_0402_1005Metric
- removed R3, R4, R6, R7: 4K7, Resistor_SMD:R_0402_1005Metric
- removed R5: 200K, Resistor_SMD:R_0402_1005Metric
- removed R8: 1K21, Resistor_SMD:R_0402_1005Metric
- removed SW2: SW_DIP_x06, Button_Switch_SMD:SW_DIP_SPSTx06_Slide_Omron_A6H-6101_W6.15mm_P1.27mm
- removed SW3, SW4: SW_DIP_x01, Connector_PinHeader_2.54mm:PinHeader_1x02_P2.54mm_Vertical
- removed U1: LTM4624IYPBF, spark:Analog_Devices_Inc-BGA-0-05-08-1905_Rev_C-0
- removed U2: PCA9306, Package_SO:SO-8_3.9x4.9mm_P1.27mm
- added F1: Fuse, spark:Fuse-Littelfuse-PTF-77P, F.Cu at (63.0, 61.0)
- added J101: Conn_01x01, spark:banana-plug-horizontal, F.Cu at (163.0, 134.0)
- added J102: Conn_01x01, spark:banana-plug-horizontal, F.Cu at (151.0, 134.0)
- added J103: Barrel_Jack, spark:PJ1-021-SMT-TR, F.Cu at (157.0, 145.7)
- added J201: Conn_01x01, spark:banana-plug-horizontal, F.Cu at (139.0, 134.0)
- added J202: Conn_01x01, spark:banana-plug-horizontal, F.Cu at (127.0, 134.0)
- added J203: Barrel_Jack, spark:PJ1-021-SMT-TR, F.Cu at (133.0, 145.7)
- added J301: Conn_01x01, spark:banana-plug-horizontal, F.Cu at (115.0, 134.0)
- added J302: Conn_01x01, spark:banana-plug-horizontal, F.Cu at (103.0, 134.0)
- added J303: Barrel_Jack, spark:PJ1-021-SMT-TR, F.Cu at (109.0, 145.7)
- added J401: Conn_01x01, spark:banana-plug-horizontal, F.Cu at (91.0, 134.0)
- added J402: Conn_01x01, spark:banana-plug-horizontal, F.Cu at (79.0, 134.0)
- added J403: Barrel_Jack, spark:PJ1-021-SMT-TR, F.Cu at (85.0, 145.7)
- added J501: Conn_01x01, spark:banana-plug-horizontal, F.Cu at (67.0, 134.0)
- added J502: Conn_01x01, spark:banana-plug-horizontal, F.Cu at (55.0, 134.0)
- added J503: Barrel_Jack, spark:PJ1-021-SMT-TR, F.Cu at (61.0, 145.7)
- added J601: Conn_01x01, spark:banana-plug-horizontal, F.Cu at (43.0, 134.0)
- added J602: Conn_01x01, spark:banana-plug-horizontal, F.Cu at (31.0, 134.0)
- added J603: Barrel_Jack, spark:PJ1-021-SMT-TR, F.Cu at (37.0, 145.7)
- added K101: G5LE-1, Relay_THT:Relay_SPDT_Omron-G5LE-1, F.Cu at (157.0, 106.0)
- added K201: G5LE-1, Relay_THT:Relay_SPDT_Omron-G5LE-1, F.Cu at (133.0, 106.0)
- added K301: G5LE-1, Relay_THT:Relay_SPDT_Omron-G5LE-1, F.Cu at (109.0, 106.0)
- added K401: G5LE-1, Relay_THT:Relay_SPDT_Omron-G5LE-1, F.Cu at (85.0, 106.0)
- added K501: G5LE-1, Relay_THT:Relay_SPDT_Omron-G5LE-1, F.Cu at (61.0, 106.0)
- added K601: G5LE-1, Relay_THT:Relay_SPDT_Omron-G5LE-1, F.Cu at (37.0, 106.0)
- added Q101: BS870, Package_TO_SOT_SMD:SOT-23, F.Cu at (163.0, 101.0)
- added Q201: BS870, Package_TO_SOT_SMD:SOT-23, F.Cu at (139.0, 101.0)
- added Q301: BS870, Package_TO_SOT_SMD:SOT-23, F.Cu at (115.0, 101.0)
- added Q401: BS870, Package_TO_SOT_SMD:SOT-23, F.Cu at (91.0, 101.0)
- added Q501: BS870, Package_TO_SOT_SMD:SOT-23, F.Cu at (67.0, 101.0)
- added Q601: BS870, Package_TO_SOT_SMD:SOT-23, F.Cu at (43.0, 101.0)
- added REF**: 96Boards CE Outline Brick, spark:96Boards_CE_outline_std_brick, B.Cu at (102.0, 41.0)
- D101, D201, D301, D401, D501, D601: value ADM_LED -> D_Schottky; footprint LED_SMD:LED_0402_1005Metric -> Diode_SMD:D_0603_1608Metric
- J1, J2: value SFP+ -> Conn_01x01; footprint spark:molex-sfp-plus-747540-101 -> spark:banana-plug-horizontal
- R101, R201, R301, R401, R501, R601: value 1K -> 10K
- R102, R202, R302, R402, R502, R602: value 10K -> 1K
- REF**: footprint spark:96Boards_CE_outline_std_brick -> spark:96Boards_CE_outline_std_brick_left
- moved J1 126.3 mm to (43.0, 54.5), turned to 270 degrees
- moved J2 115.6 mm to (31.0, 54.5), turned to 270 degrees
- moved R602 70.7 mm to (44.0, 98.2)
- moved REF** 69.0 mm to (20.0, 51.5), turned to 180 degrees
- moved R502 58.0 mm to (68.0, 98.2)
- moved R402 46.2 mm to (92.0, 98.2)
- moved R302 36.0 mm to (116.0, 98.2)
- moved R202 29.1 mm to (140.0, 98.2)
- moved R102 28.1 mm to (164.0, 98.2)
- moved R101 5.51 mm to (162.5, 98.7), turned to 180 degrees
- moved R201 5.51 mm to (138.5, 98.7), turned to 180 degrees
- moved R301 5.51 mm to (114.5, 98.7), turned to 180 degrees
- moved R401 5.51 mm to (90.5, 98.7), turned to 180 degrees
- moved R501 5.51 mm to (66.5, 98.7), turned to 180 degrees
- moved R601 5.51 mm to (42.5, 98.7), turned to 180 degrees
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Connections:
- D101 pad 1: SFP0_ADM_LED -> +12V
- D201 pad 1: SFP1_ADM_LED -> +12V
- D301 pad 1: SFP2_ADM_LED -> +12V
- D401 pad 1: SFP3_ADM_LED -> +12V
- D501 pad 1: SFP4_ADM_LED -> +12V
- D601 pad 1: SFP5_ADM_LED -> +12V
- J1 pad 1: GND -> +12V
- R101 pad 1: +3V3 -> Net-(Q101-Pad1)
- R101 pad 2: Net-(D101-Pad2) -> GND
- R102 pad 1: +3V3 -> GPIO_E
- R102 pad 2: SFP0_MOD_ABS -> Net-(Q101-Pad1)
- R201 pad 1: +3V3 -> Net-(Q201-Pad1)
- R201 pad 2: Net-(D201-Pad2) -> GND
- R202 pad 1: +3V3 -> GPIO_F
- R202 pad 2: SFP1_MOD_ABS -> Net-(Q201-Pad1)
- R301 pad 1: +3V3 -> Net-(Q301-Pad1)
- R301 pad 2: Net-(D301-Pad2) -> GND
- R302 pad 1: +3V3 -> GPIO_C
- R302 pad 2: SFP2_MOD_ABS -> Net-(Q301-Pad1)
- R401 pad 1: +3V3 -> Net-(Q401-Pad1)
- R401 pad 2: Net-(D401-Pad2) -> GND
- R402 pad 1: +3V3 -> GPIO_D
- R402 pad 2: SFP3_MOD_ABS -> Net-(Q401-Pad1)
- R501 pad 1: +3V3 -> Net-(Q501-Pad1)
- R501 pad 2: Net-(D501-Pad2) -> GND
- R502 pad 1: +3V3 -> GPIO_A
- R502 pad 2: SFP4_MOD_ABS -> Net-(Q501-Pad1)
- R601 pad 1: +3V3 -> Net-(Q601-Pad1)
- R601 pad 2: Net-(D601-Pad2) -> GND
- R602 pad 1: +3V3 -> GPIO_B
- R602 pad 2: SFP5_MOD_ABS -> Net-(Q601-Pad1)
- REF** pad 1: CHASSIS -> (no net) (x2)
Routing:
- net GND: track 1508.2 -> 48.6 mm, vias 151 -> 23
- net +3V3: track 359.2 -> 0.00 mm, vias 57 -> 0
- net CSI0_C+: track 274.4 -> 0.00 mm
- net CSI0_C-: track 271.4 -> 0.00 mm
- net CSI0_D3+: track 249.2 -> 0.00 mm, vias 2 -> 0
- net CSI0_D3-: track 247.8 -> 0.00 mm, vias 2 -> 0
- net CSI0_D1+: track 241.5 -> 0.00 mm
- net CSI0_D1-: track 238.5 -> 0.00 mm
- net GPIO_B: track 5.35 -> 232.1 mm
- net CSI0_D2+: track 217.0 -> 0.00 mm
- net CSI0_D2-: track 215.5 -> 0.00 mm
- net CSI1_D0+: track 205.2 -> 0.00 mm
- net CHASSIS: track 202.4 -> 0.00 mm
- net CSI1_D0-: track 202.3 -> 0.00 mm
- net GPIO_A: track 14.6 -> 209.6 mm
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- added copper zone on In2.Cu, net +12V
- added copper zone on F.Cu, net Net-(J101-Pad1)
- added copper zone on In2.Cu, net Net-(J101-Pad1)
- added copper zone on F.Cu, net Net-(J201-Pad1)
- added copper zone on In2.Cu, net Net-(J201-Pad1)
- added copper zone on F.Cu, net Net-(J301-Pad1)
- added copper zone on In2.Cu, net Net-(J301-Pad1)
- added copper zone on F.Cu, net Net-(J401-Pad1)
- added copper zone on In2.Cu, net Net-(J401-Pad1)
- added copper zone on F.Cu, net Net-(J501-Pad1)
- added copper zone on In2.Cu, net Net-(J501-Pad1)
- added copper zone on F.Cu, net Net-(J601-Pad1)
- added copper zone on In2.Cu, net Net-(J601-Pad1)
- removed copper zone on F.Cu, net +3V3
- removed copper zone on In2.Cu, net +3V3
- removed copper zone on F.Cu, net SYS_DCIN
Other:
- board text added: "P/N: SPARK-PDU V1 REV: 1"
- board text removed: "9"
- board text removed: ":"
- board text removed: "P/N"
- board text removed: "REV"
- board text removed: "SPARK-V2"

Commit message: spark-pdu-pi-1.0-1
Parts:
- removed the ? at (192.0, 45.0)
- removed the ? at (250.0, 45.0)
- removed P1: CONN_02X20, spark:Pin_Header_SMD_2x20_Pitch2mm
- removed P2: Conn_02x20_Odd_Even, spark:Socket_Strip_SMD_2x20_Pitch2mm
- removed the REF** at (273.0, 150.0)
- added ?: , spark:mount_hole, F.Cu at (269.0, 68.5)
- added ?: , spark:mount_hole, F.Cu at (269.0, 126.5)
- added ?: , spark:mount_hole, F.Cu at (197.0, 68.5)
- added ?: , spark:mount_hole, F.Cu at (197.0, 126.5)
- added ?: , spark:mount_hole, F.Cu at (246.0, 126.5)
- added ?: , spark:mount_hole, F.Cu at (246.0, 68.5)
- added C1: 2.2uF, Capacitor_SMD:C_0603_1608Metric, F.Cu at (130.0, 46.5)
- added C2: 2.2uF, Capacitor_SMD:C_0603_1608Metric, F.Cu at (125.3, 49.5)
- added C3: 22uF, Capacitor_SMD:C_0805_2012Metric, F.Cu at (139.6, 49.2)
- added C4: 22uF, Capacitor_SMD:C_0805_2012Metric, F.Cu at (139.6, 47.2)
- added C5: 0.1uF, Capacitor_SMD:C_0402_1005Metric, F.Cu at (135.0, 50.4)
- added C6: 10uF, Capacitor_SMD:C_0805_2012Metric, F.Cu at (125.1, 51.7)
- added C8: 22nF, Capacitor_SMD:C_0402_1005Metric, F.Cu at (130.5, 53.2)
- added C9: 0.1uF, Capacitor_SMD:C_0402_1005Metric, F.Cu at (134.2, 52.1)
- added L1: 10uH, Inductor_SMD:L_1210_3225Metric, F.Cu at (135.5, 48.3)
- added P5: Conn_02x20_Odd_Even, spark:PinSocket_2x20_P2.54mm_Vertical_1_04mm, F.Cu at (270.3, 73.4)
- added R5: 4.7K, Capacitor_SMD:C_0402_1005Metric, F.Cu at (134.2, 53.1)
- added R6: 105K, Resistor_SMD:R_0402_1005Metric, F.Cu at (134.2, 54.1)
- added R7: 22.6K, Resistor_SMD:R_0402_1005Metric, F.Cu at (134.2, 55.1)
- added U1: MAX17574, Package_DFN_QFN:QFN-24-1EP_4x5mm_P0.5mm_EP2.65x3.65mm, F.Cu at (130.0, 50.0)
- REF**: value 96Boards CE Outline Brick -> 96Boards CE Outline Brick Top; footprint spark:96Boards_CE_outline_std_brick -> spark:96Boards_CE_outline_std_brick_top
- moved REF** 131.8 mm to (184.6, 146.2)
- moved REF** 100.7 mm to (273.0, 95.0), turned to 180 degrees
Routing:
- net PWR_BTN_N: track 145.6 -> 237.8 mm, vias 1 -> 0
- net GPIO_E: track 105.6 -> 188.6 mm
- net GPIO_F: track 126.9 -> 208.5 mm
- net GPIO_D: track 180.4 -> 258.2 mm
- net GPIO_C: track 158.6 -> 231.4 mm
- net GPIO_A: track 209.6 -> 280.3 mm
- net GPIO_B: track 232.1 -> 302.7 mm
- net SYS_DCIN: track 30.0 -> 10.6 mm, vias 6 -> 7
- net I2C1_SDA: track 15.8 -> 0.00 mm
- net +1V8: track 15.2 -> 0.00 mm, vias 2 -> 0
- net UART1_TX: track 14.6 -> 0.00 mm
- net UART1_RX: track 14.6 -> 0.00 mm
- net UART0_TX: track 14.6 -> 0.00 mm
- net UART0_RX: track 14.6 -> 0.00 mm
- net UART0_RTS: track 14.6 -> 0.00 mm
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- added copper zone on F.Cu, net +5V
- added copper zone on In2.Cu, net +5V
- added copper zone on F.Cu, net Net-(C5-Pad1)
- added copper zone on F.Cu, net SYS_DCIN
Other:
- outline, holes or cut-outs redrawn
- board text added: "12V -> 5V (3A max)"
- board text added: "P/N: SPARK-PDU-PI V1 REV: 1"
- board text removed: "P/N: SPARK-PDU V1 REV: 1"

Commit message: spark-pdu-pi-1-2
Parts:
- J1: footprint spark:banana-plug-horizontal -> spark:banana-plug-horizontal-red
- J2: footprint spark:banana-plug-horizontal -> spark:banana-plug-horizontal-black
- P5: footprint spark:PinSocket_2x20_P2.54mm_Vertical_1_04mm -> spark:PinHeader_2x20_P2.54mm_Vertical_1_04mm
- moved REF** 14.3 mm to (183.0, 132.0)
Other:
- board text added: "P/N: SPARK-PDU-PI V1 REV: 2"
- board text removed: "P/N: SPARK-PDU-PI V1 REV: 1"

Commit message: spark-pdu-pi-1-3
Parts:
- removed C1, C2: 2.2uF, Capacitor_SMD:C_0603_1608Metric
- removed C3, C4: 22uF, Capacitor_SMD:C_0805_2012Metric
- removed C5, C9: 0.1uF, Capacitor_SMD:C_0402_1005Metric
- removed C6: 10uF, Capacitor_SMD:C_0805_2012Metric
- removed C8: 22nF, Capacitor_SMD:C_0402_1005Metric
- removed L1: 10uH, Inductor_SMD:L_1210_3225Metric
- removed R5: 4.7K, Capacitor_SMD:C_0402_1005Metric
- removed R6: 105K, Resistor_SMD:R_0402_1005Metric
- removed R7: 22.6K, Resistor_SMD:R_0402_1005Metric
- removed the REF** at (102.0, 41.0)
- removed U1: MAX17574, Package_DFN_QFN:QFN-24-1EP_4x5mm_P0.5mm_EP2.65x3.65mm
- added J3: Conn_02x06_Odd_Even, spark:Socket_Strip_SMD_2x6_Pitch2mm, F.Cu at (249.0, 137.0)
- added J4: Conn_02x06_Odd_Even, spark:Socket_Strip_SMD_2x6_Pitch2mm, F.Cu at (268.0, 137.0)
- P5: value Conn_02x20_Odd_Even -> Raspberry_Pi_2_3
- moved P5 7.56 mm to (262.7, 72.9)
- moved ? 5.02 mm to (241.0, 68.0)
- moved ? 5.02 mm to (241.0, 126.0)
- moved ? 5.02 mm to (192.0, 126.0)
- moved ? 5.02 mm to (192.0, 68.0)
- moved ? 5.02 mm to (264.0, 126.0)
- moved ? 5.02 mm to (264.0, 68.0)
Connections:
- net GPIO_A renamed PORT5
- net GPIO_B renamed PORT6
- P5 pad 1: +5V -> +3V3
- P5 pad 15: GPIO_D -> PORT3
- P5 pad 16: GPIO_C -> PORT4
- P5 pad 17: (no net) -> +3V3
- P5 pad 18: GPIO_F -> (no net)
- P5 pad 2: (no net) -> +5V
- P5 pad 22: GPIO_E -> (no net)
- P5 pad 29: PWR_BTN_N -> (no net)
- P5 pad 3: +5V -> (no net)
- P5 pad 36: (no net) -> PORT2
- P5 pad 37: (no net) -> PORT1
- P5 pad 4: (no net) -> +5V
- P5 pad 40: (no net) -> RESET_BTN
- R102 pad 1: GPIO_E -> PORT1
- R202 pad 1: GPIO_F -> PORT2
- R302 pad 1: GPIO_C -> PORT3
- R402 pad 1: GPIO_D -> PORT4
- SW1 pad 2: PWR_BTN_N -> RESET_BTN
Routing:
- net GPIO_D: track 258.2 -> 0.00 mm
- net PORT3: track 0.00 -> 254.6 mm
- net PORT4: track 0.00 -> 252.8 mm
- net RESET_BTN: track 0.00 -> 245.3 mm
- net PWR_BTN_N: track 237.8 -> 0.00 mm
- net GPIO_C: track 231.4 -> 0.00 mm
- net PORT2: track 0.00 -> 227.9 mm
- net GPIO_F: track 208.5 -> 0.00 mm
- net PORT1: track 0.00 -> 203.7 mm
- net GPIO_E: track 188.6 -> 0.00 mm
- net GND: track 37.0 -> 29.4 mm
- net PORT5: track 280.3 -> 273.2 mm
- net PORT6: track 302.7 -> 295.7 mm
- net +5V: track 6.20 -> 0.00 mm, vias 5 -> 6
- net Net-(R6-Pad2): track 4.82 -> 0.00 mm
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- removed copper zone on F.Cu, net Net-(C5-Pad1)
Other:
- outline, holes or cut-outs redrawn
- board text added: "12V -> 5V"
- board text added: "27x16 mm"
- board text added: "P/N: SPARK-PDU-PI V1 REV: 3"
- board text removed: "12V -> 5V (3A max)"
- board text removed: "P/N: SPARK-PDU-PI V1 REV: 2"

Commit message: spark-pdu-pi-1-4
Connections:
- D101 pad 1: +12V -> SYS_DCIN
- D201 pad 1: +12V -> SYS_DCIN
- D301 pad 1: +12V -> SYS_DCIN
- D401 pad 1: +12V -> SYS_DCIN
- D501 pad 1: +12V -> SYS_DCIN
- D601 pad 1: +12V -> SYS_DCIN
- F1 pad 2: +12V -> IN
- J1 pad 1: +12V -> IN
- K101 pad 1: +12V -> IN
- K101 pad 2: +12V -> SYS_DCIN
- K201 pad 1: +12V -> IN
- K201 pad 2: +12V -> SYS_DCIN
- K301 pad 1: +12V -> IN
- K301 pad 2: +12V -> SYS_DCIN
- K401 pad 1: +12V -> IN
- K401 pad 2: +12V -> SYS_DCIN
- K501 pad 1: +12V -> IN
- K501 pad 2: +12V -> SYS_DCIN
- K601 pad 1: +12V -> IN
- K601 pad 2: +12V -> SYS_DCIN
Routing:
- net SYS_DCIN: track 10.6 -> 490.2 mm, vias 10 -> 11
- net +12V: track 24.0 -> 0.00 mm
- net GND: track 29.4 -> 31.5 mm, vias 23 -> 24
- added copper zone on In2.Cu, net IN
- removed copper zone on In2.Cu, net +12V
Other:
- board text added: "P/N: SPARK-PDU-PI V1 REV: 4"
- board text removed: "P/N: SPARK-PDU-PI V1 REV: 3"

Commit message: spark-relay-actuator-pi-1-1
Parts:
- removed the ? at (58.5, 76.6)
- removed D401, D501, D601: D_Schottky, Diode_SMD:D_0603_1608Metric
- removed F1: Fuse, spark:Fuse-Littelfuse-PTF-77P
- removed J1: Conn_01x01, spark:banana-plug-horizontal-red
- removed J2: Conn_01x01, spark:banana-plug-horizontal-black
- removed J401, J402, J501, J502, J601, J602: Conn_01x01, spark:banana-plug-horizontal
- removed J403, J503, J603: Barrel_Jack, spark:PJ1-021-SMT-TR
- removed K401, K501, K601: G5LE-1, Relay_THT:Relay_SPDT_Omron-G5LE-1
- removed Q401, Q501, Q601: BS870, Package_TO_SOT_SMD:SOT-23
- removed R401, R501, R601: 10K, Resistor_SMD:R_0402_1005Metric
- removed R402, R502, R602: 1K, Resistor_SMD:R_0402_1005Metric
- removed the REF** at (273.0, 95.0)
- removed the REF** at (20.0, 140.5)
- removed the REF** at (20.0, 51.5)
- removed the REF** at (101.0, 95.0)
- removed the REF** at (183.0, 132.0)
- added REF**: Hole_2.5MM, spark:Hole_2.5MM, F.Cu at (438.8, 48.8)
- added REF**: Hole_2.5MM, spark:Hole_2.5MM, F.Cu at (352.8, 48.8)
- added REF**: Hole_2.5MM, spark:Hole_2.5MM, F.Cu at (189.8, 62.8)
- added REF**: Hole_2.5MM, spark:Hole_2.5MM, F.Cu at (189.8, 134.8)
- J101, J102, J201, J202, J301, J302: footprint spark:banana-plug-horizontal -> spark:banana-plug-horizontal-black
- J103, J203, J303: value Barrel_Jack -> Conn_01x01; footprint spark:PJ1-021-SMT-TR -> spark:banana-plug-horizontal-black
- REF**: moved to F.Cu
- moved J103 141.0 mm to (49.0, 55.0), turned to 270 degrees
- moved R102 135.7 mm to (29.0, 111.7), turned to 90 degrees
- moved Q101 133.2 mm to (30.0, 108.9), turned to 90 degrees
- moved R101 132.6 mm to (30.5, 111.2), turned to 0 degrees
- moved J101 126.0 mm to (37.0, 134.0)
- moved D101 122.9 mm to (35.0, 108.0), turned to 180 degrees
- moved K101 108.0 mm to (49.0, 106.0)
- moved J203 97.6 mm to (97.0, 55.0), turned to 270 degrees
- moved J303 97.6 mm to (145.0, 55.0), turned to 270 degrees
- moved J10 92.0 mm to (169.0, 45.0)
- moved J102 90.0 mm to (61.0, 134.0)
- moved R202 64.4 mm to (77.0, 111.7), turned to 90 degrees
- moved Q201 61.5 mm to (78.0, 108.9), turned to 90 degrees
- moved R201 61.3 mm to (78.5, 111.2), turned to 0 degrees
- moved J201 54.0 mm to (85.0, 134.0)
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Connections:
- J102 pad 1: GND -> Net-(J102-Pad1)
- J103 pad 1: Net-(J101-Pad1) -> IN1
- J202 pad 1: GND -> Net-(J202-Pad1)
- J203 pad 1: Net-(J201-Pad1) -> IN2
- J302 pad 1: GND -> Net-(J302-Pad1)
- J303 pad 1: Net-(J301-Pad1) -> IN3
- K101 pad 1: IN -> IN1
- K101 pad 4: (no net) -> Net-(J102-Pad1)
- K201 pad 1: IN -> IN2
- K201 pad 4: (no net) -> Net-(J202-Pad1)
- K301 pad 1: IN -> IN3
- K301 pad 4: (no net) -> Net-(J302-Pad1)
- P5 pad 11: PORT6 -> PORT3
- P5 pad 13: PORT5 -> PORT2
- P5 pad 15: PORT3 -> (no net)
- P5 pad 16: PORT4 -> PORT1
- P5 pad 36: PORT2 -> (no net)
- P5 pad 37: PORT1 -> (no net)
Routing:
- net PORT6: track 295.7 -> 0.00 mm
- net PORT5: track 273.2 -> 0.00 mm
- net SYS_DCIN: track 490.2 -> 218.4 mm
- net PORT4: track 252.8 -> 0.00 mm
- net GND: track 31.5 -> 187.3 mm, vias 24 -> 21
- net PORT1: track 203.7 -> 323.6 mm
- net IN2: track 0.00 -> 51.0 mm
- net IN1: track 0.00 -> 51.0 mm
- net IN3: track 0.00 -> 51.0 mm
- net PORT2: track 227.9 -> 271.3 mm
- net PORT3: track 254.6 -> 220.8 mm
- net Net-(D301-Pad2): track 10.4 -> 28.9 mm
- net Net-(D201-Pad2): track 10.4 -> 28.9 mm
- net Net-(D101-Pad2): track 10.4 -> 28.9 mm
- net Net-(D601-Pad2): track 10.4 -> 0.00 mm
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- added copper zone on B.Cu, net IN1
- added copper zone on B.Cu, net IN2
- added copper zone on B.Cu, net IN3
- added copper zone on B.Cu, net Net-(J101-Pad1)
- added copper zone on B.Cu, net Net-(J102-Pad1)
- added copper zone on B.Cu, net Net-(J201-Pad1)
- added copper zone on B.Cu, net Net-(J202-Pad1)
- added copper zone on B.Cu, net Net-(J301-Pad1)
- added copper zone on B.Cu, net Net-(J302-Pad1)
- removed copper zone on In2.Cu, net IN
- removed copper zone on F.Cu, net Net-(J101-Pad1)
- removed copper zone on In2.Cu, net Net-(J101-Pad1)
- removed copper zone on F.Cu, net Net-(J201-Pad1)
- removed copper zone on In2.Cu, net Net-(J201-Pad1)
- removed copper zone on F.Cu, net Net-(J301-Pad1)
- removed copper zone on In2.Cu, net Net-(J301-Pad1)
- removed copper zone on F.Cu, net Net-(J401-Pad1)
- removed copper zone on In2.Cu, net Net-(J401-Pad1)
- removed copper zone on F.Cu, net Net-(J501-Pad1)
- removed copper zone on In2.Cu, net Net-(J501-Pad1)
- removed copper zone on F.Cu, net Net-(J601-Pad1)
- removed copper zone on In2.Cu, net Net-(J601-Pad1)
Other:
- board text added: "P/N: SPARK-RELAY-ACTUATOR-PI V1 REV: 1"
- board text removed: "P/N: SPARK-PDU-PI V1 REV: 4"
