File: board/spark.kicad_pcb (KiCad board)
At the start: 4 copper layers, 257 x 109 mm, 40 parts, among them J10 Barrel_Jack, J101 Conn_01x01, J102 Conn_01x01, J103 Conn_01x01, J201 Conn_01x01, J202 Conn_01x01, J203 Conn_01x01, J3 Conn_02x06_Odd_Even, J301 Conn_01x01, J302 Conn_01x01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

Commit message: spark-relay-actuator-pi-1-2
Parts:
- removed the REF** at (189.8, 62.8)
- added ?: , spark:lightside-instruments-logo, F.Cu at (226.0, 45.0)
- added REF**: Hole_2.5MM, spark:Hole_2.5MM, F.Cu at (189.8, 103.2)
- added REF**: Hole_2.5MM, spark:Hole_2.5MM, F.Cu at (189.8, 48.2)
- moved J103 2.00 mm to (49.0, 57.0)
- moved J203 2.00 mm to (97.0, 57.0)
- moved J303 2.00 mm to (145.0, 57.0)
Other:
- board text added: "P/N: SPARK-RELAY-ACTUATOR-PI V1 REV: 2"
- board text removed: "P/N: SPARK-RELAY-ACTUATOR-PI V1 REV: 1"

Commit message: spark-relay-actuator-pi-1-3
Parts:
- added D102: LED, Diode_SMD:D_0603_1608Metric, F.Cu at (49.0, 149.0)
- added D202: LED, Diode_SMD:D_0603_1608Metric, F.Cu at (97.2, 149.0)
- added D302: LED, Diode_SMD:D_0603_1608Metric, F.Cu at (145.0, 149.0)
- added R103: 1K, Resistor_SMD:R_0402_1005Metric, F.Cu at (50.0, 147.0)
- added R203: 1K, Resistor_SMD:R_0402_1005Metric, F.Cu at (98.0, 147.0)
- added R303: 1K, Resistor_SMD:R_0402_1005Metric, F.Cu at (146.0, 147.0)
Routing:
- net SYS_DCIN: track 218.4 -> 345.5 mm, vias 11 -> 14
- net Net-(D301-Pad2): track 28.9 -> 69.0 mm, vias 0 -> 1
- net Net-(D201-Pad2): track 28.9 -> 69.0 mm, vias 0 -> 1
- net Net-(D101-Pad2): track 28.9 -> 69.0 mm, vias 0 -> 1
- net Net-(D302-Pad1): track 0.00 -> 1.30 mm
- net Net-(D202-Pad1): track 0.00 -> 1.30 mm
- net Net-(D102-Pad1): track 0.00 -> 1.30 mm
- net GND: track 187.3 -> 186.5 mm
Other:
- board text added: "P/N: SPARK-RELAY-ACTUATOR-PI V1 REV: 3"
- board text removed: "P/N: SPARK-RELAY-ACTUATOR-PI V1 REV: 2"

Commit message: spark-relay-actuator-pi-2-1
Parts:
- removed the ? at (241.0, 68.0)
- removed the ? at (241.0, 126.0)
- removed the ? at (192.0, 126.0)
- removed the ? at (192.0, 68.0)
- removed the ? at (226.0, 45.0)
- removed the REF** at (189.8, 103.2)
- removed the REF** at (438.8, 48.8)
- removed the REF** at (352.8, 48.8)
- removed the REF** at (189.8, 48.2)
- removed the REF** at (189.8, 134.8)
- added ?: , spark:Hole_2.5MM, F.Cu at (210.5, 45.0)
- added ?: , spark:lightside-instruments-logo-silks, F.Cu at (134.5, 68.2)
- added ?: , spark:mount_hole, F.Cu at (159.0, 76.0)
- added ?: , spark:mount_hole, F.Cu at (110.0, 76.0)
- added REF**: Hole_2.5MM, spark:Hole_2.5MM, F.Cu at (38.5, 107.5)
- moved P5 245.6 mm to (18.2, 49.4)
- moved ? 245.6 mm to (19.5, 102.5)
- moved ? 245.6 mm to (19.5, 44.5)
- moved J3 226.9 mm to (33.5, 66.0)
- moved J4 226.9 mm to (52.5, 66.0)
- moved SW1 139.3 mm to (41.8, 123.0)
- moved J10 129.5 mm to (39.5, 45.0)
- moved D101 44.5 mm to (72.5, 84.0)
- moved D102 44.5 mm to (86.5, 125.0)
- moved D201 44.5 mm to (120.5, 84.0)
- moved D202 44.5 mm to (134.7, 125.0)
- moved D301 44.5 mm to (168.5, 84.0)
- moved D302 44.5 mm to (182.5, 125.0)
- moved J101 44.5 mm to (74.5, 110.0)
- moved J102 44.5 mm to (98.5, 110.0)
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Connections:
- P5 pad 11: PORT3 -> PORT1
- P5 pad 16: PORT1 -> PORT3
Routing:
- net PORT1: track 323.6 -> 70.0 mm
- net RESET_BTN: track 235.2 -> 32.2 mm
- net PORT2: track 271.3 -> 113.7 mm
- net PORT3: track 220.8 -> 158.2 mm
- net IN2: track 51.0 -> 25.0 mm
- net IN3: track 51.0 -> 25.0 mm
- net IN1: track 51.0 -> 25.0 mm
- net GND: track 186.5 -> 195.7 mm, vias 21 -> 20
- added copper zone on B.Cu, net +5V
- removed copper zone on In2.Cu, net +5V
Other:
- board size 257 x 109 mm -> 198.5 x 85 mm
- board text added: "1"
- board text added: "2"
- board text added: "3"
- board text added: "A"
- board text added: "B"
- board text added: "P/N: SPARK-RELAY-ACTUATOR-PI V2 REV: 1"
- board text removed: "P/N: SPARK-RELAY-ACTUATOR-PI V1 REV: 3"
